File: hardware/YABR_Bot/YABR_Bot.kicad_pcb (KiCad board)
At the start: 2 copper layers, 110 x 85 mm, 22 parts, among them J1 SERVO, J2 SERVO, J3 Conn_01x02_Socket, M1 Stepper_Motor_bipolar, M2 Stepper_Motor_bipolar, U2 DRV8825, U3 DRV8825, U4 DCDC_StepDown_LM2596, U5 ESP32-DevKitC

Commit message: Update Hardware to V2
Parts:
- removed the R1 at (104.0, 71.0)
- removed SV1, SV2: MSI1, yabr-main-4:MA03-2
- added D3: LED, LED_THT:LED_D3.0mm, F.Cu at (74.9, 34.3)
- added D4: LED, LED_THT:LED_D3.0mm, F.Cu at (68.6, 34.3)
- added FID1: Fiducial, Fiducial:Fiducial_1.5mm_Mask3mm, F.Cu at (25.0, 22.0)
- added FID2: Fiducial, Fiducial:Fiducial_1.5mm_Mask3mm, F.Cu at (25.0, 97.0)
- added FID3: Fiducial, Fiducial:Fiducial_1.5mm_Mask3mm, F.Cu at (125.0, 97.0)
- added H1: MountingHole, MountingHole:MountingHole_3.2mm_M3, F.Cu at (25.0, 22.0)
- added H2: MountingHole, MountingHole:MountingHole_3.2mm_M3, F.Cu at (25.0, 97.0)
- added H3: MountingHole, MountingHole:MountingHole_3.2mm_M3, F.Cu at (125.0, 97.0)
- added H4: MountingHole, MountingHole:MountingHole_3.2mm_M3, F.Cu at (125.0, 22.0)
- added H5: MountingHole, MountingHole:MountingHole_3.2mm_M3, F.Cu at (67.7, 84.1)
- added H6: MountingHole, MountingHole:MountingHole_3.2mm_M3, F.Cu at (84.7, 84.1)
- added R6: 82, Resistor_THT:R_Axial_DIN0309_L9.0mm_D3.2mm_P12.70mm_Horizontal, F.Cu at (69.8, 53.3)
- added R7: 82, Resistor_THT:R_Axial_DIN0309_L9.0mm_D3.2mm_P12.70mm_Horizontal, F.Cu at (66.0, 53.3)
- added R8: 1K1, Resistor_THT:R_Axial_DIN0309_L9.0mm_D3.2mm_P12.70mm_Horizontal, F.Cu at (108.0, 29.2)
- added R9: 1K1, Resistor_THT:R_Axial_DIN0309_L9.0mm_D3.2mm_P12.70mm_Horizontal, F.Cu at (92.7, 29.2)
- added SW1: SW_Push, Button_Switch_THT:SW_PUSH_6mm_H9.5mm, F.Cu at (111.0, 20.8)
- added SW2: SW_Push, Button_Switch_THT:SW_PUSH_6mm_H9.5mm, F.Cu at (102.2, 25.2)
- D1, D2: footprint LED_SMD:LED_1206_3216Metric_Pad1.42x1.75mm_HandSolder -> LED_THT:LED_D3.0mm
- R1: renamed from R5; footprint yabr-main-4:0207_10 -> Resistor_THT:R_Axial_DIN0309_L9.0mm_D3.2mm_P12.70mm_Horizontal
- R2: renamed from R6; footprint yabr-main-4:0207_10 -> Resistor_THT:R_Axial_DIN0309_L9.0mm_D3.2mm_P12.70mm_Horizontal
- R3: value 4k7 -> 4K7; footprint yabr-main-4:0207_10 -> Resistor_THT:R_Axial_DIN0309_L9.0mm_D3.2mm_P12.70mm_Horizontal
- R4: renamed from R2; value 160 -> 1K1; footprint Resistor_SMD:R_1206_3216Metric_Pad1.30x1.75mm_HandSolder -> Resistor_THT:R_Axial_DIN0309_L9.0mm_D3.2mm_P12.70mm_Horizontal
- R5: renamed from R4; value 160 -> 1K1; footprint Resistor_SMD:R_1206_3216Metric_Pad1.30x1.75mm_HandSolder -> Resistor_THT:R_Axial_DIN0309_L9.0mm_D3.2mm_P12.70mm_Horizontal
- moved R3 38.1 mm to (69.8, 66.7), turned to 0 degrees
- moved J3 34.6 mm to (83.0, 24.0)
- moved J2 32.1 mm to (74.0, 24.0)
- moved U1 29.6 mm to (60.2, 24.5), turned to -90 degrees
- moved R2 23.5 mm to (37.0, 29.0), turned to -90 degrees
- moved R4 21.1 mm to (90.8, 97.8), turned to 90 degrees
- moved R5 14.7 mm to (39.4, 70.1), turned to 180 degrees
- moved D1 10.5 mm to (98.4, 77.5), turned to 180 degrees
- moved D2 9.26 mm to (26.7, 78.7)
- moved R1 6.78 mm to (37.0, 45.0)
- moved C1 1.37 mm to (45.7, 96.5)
- moved J1 1.34 mm to (31.8, 49.5)
- moved U2 1.29 mm to (82.1, 59.7)
- moved C2 1.26 mm to (116.8, 96.5)
- moved JP1 0.23 mm to (76.2, 71.1)
- renumbered J3 to J1, J1 to J2, J2 to J3, U4 to U1, U5 to U2, U2 to U3, U3 to U4
Connections:
- net /SDL renamed /SDA
- JP1 pad 1: +5V -> +3V3
- JP1 pad 8: /INT -> Net-(U2-GPIO23)
- R3 pad 1: Net-(R3-Pad1) -> /AD0
- R3 pad 2: +5V -> GND
- R4 pad 1: +5V -> VMOT
- R5 pad 1: +5V -> VMOT
- U2 pad 1: unconnected-(U5-3V3-Pad1) -> +3V3
- U2 pad 10: unconnected-(U5-DAC_2/ADC2_CH9/GPIO26-Pad10) -> /STEP_SELECT_M0
- U2 pad 11: unconnected-(U5-ADC2_CH7/GPIO27-Pad11) -> /STEP_ENABLE
- U2 pad 20: unconnected-(U5-SD_CLK/GPIO6-Pad20) -> Net-(U2-SD_CLK/GPIO6)
- U2 pad 21: unconnected-(U5-SD_DATA0/GPIO7-Pad21) -> Net-(U2-SD_DATA0/GPIO7)
- U2 pad 30: unconnected-(U5-GPIO18-Pad30) -> Net-(D4-K)
- U2 pad 31: unconnected-(U5-GPIO19-Pad31) -> Net-(D3-K)
- U2 pad 37: unconnected-(U5-GPIO23-Pad37) -> Net-(U2-GPIO23)
- U2 pad 8: unconnected-(U5-32K_XN/GPIO33/ADC1_CH5-Pad8) -> /STEP_SELECT_M2
- U2 pad 9: unconnected-(U5-DAC_1/ADC2_CH8/GPIO25-Pad9) -> /STEP_SELECT_M1
- U3 pad 10: Net-(U2-M0) -> /STEP_SELECT_M0
- U3 pad 11: Net-(U2-M1) -> /STEP_SELECT_M1
- U3 pad 12: Net-(U2-M2) -> /STEP_SELECT_M2
- U3 pad 13: Net-(U2-RST) -> unconnected-(U3-RST-Pad13)
- U3 pad 14: Net-(U2-RST) -> unconnected-(U3-SLP-Pad14)
- U3 pad 9: unconnected-(U2-EN-Pad9) -> /STEP_ENABLE
- U4 pad 10: Net-(U3-M0) -> /STEP_SELECT_M0
- U4 pad 11: Net-(U3-M1) -> /STEP_SELECT_M1
- U4 pad 12: Net-(U3-M2) -> /STEP_SELECT_M2
- U4 pad 13: Net-(U3-RST) -> unconnected-(U4-RST-Pad13)
- U4 pad 14: Net-(U3-RST) -> unconnected-(U4-SLP-Pad14)
- U4 pad 9: unconnected-(U3-EN-Pad9) -> /STEP_ENABLE
Routing:
- net GND: track 1.35 -> 429.8 mm, vias 0 -> 2
- net +3V3: track 0.00 -> 116.1 mm, vias 0 -> 4
- net +5V: track 254.1 -> 138.2 mm, vias 1 -> 3
- net /STEP_SELECT_M2: track 0.00 -> 98.8 mm, vias 0 -> 3
- net /STEP_SELECT_M1: track 0.00 -> 98.0 mm, vias 0 -> 3
- net /STEP_SELECT_M0: track 0.00 -> 97.1 mm, vias 0 -> 3
- net /STEP_ENABLE: track 0.00 -> 96.2 mm, vias 0 -> 3
- net Net-(U2-GPIO23): track 0.00 -> 53.6 mm, vias 0 -> 2
- net Net-(D3-K): track 0.00 -> 47.8 mm
- net Net-(D4-K): track 0.00 -> 47.3 mm
- net /VSENS: track 65.0 -> 105.2 mm, vias 0 -> 2
- net Net-(U2-SD_DATA0/GPIO7): track 0.00 -> 37.8 mm
- net Net-(U2-SD_CLK/GPIO6): track 0.00 -> 30.2 mm
- net VMOT: track 184.1 -> 211.3 mm, vias 0 -> 2
- net /SERVO2: track 46.0 -> 69.8 mm, vias 0 -> 2
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Other:
- outline, holes or cut-outs redrawn
- board text added: "Christopher Kösters Oliver Westermann Campuswoche 2023"
- board text removed: "Campuswoche 2023"
- board text removed: "SERVO1"
- board text removed: "SERVO2"
- board text removed: "by Christopher Kösters"
