File: hardware/YABR_Bot/YABR_Bot.kicad_sch (KiCad schematic)
At the start: 22 parts, among them J3 Conn_01x02_Socket, J6 SERVO, J7 SERVO, M1 Stepper_Motor_bipolar, M2 Stepper_Motor_bipolar, U2 DRV8825, U3 DRV8825, U4 DCDC_StepDown_LM2596, U5 ESP32-DevKitC

Commit message: Update Hardware to V2
Parts:
- removed R10 (x2): 4k7, yabr-main-4:0207_10, symbol yabr-main-4-eagle-import:R-EU_0207/10
- removed SV2 (x2): MSI1, yabr-main-4:MA03-2, symbol yabr-main-4-eagle-import:MA03-2
- added D3, D4: LED, LED_THT:LED_D3.0mm, symbol Device:LED
- added FID1, FID2, FID3: Fiducial, Fiducial:Fiducial_1.5mm_Mask3mm, symbol Mechanical:Fiducial
- added H1, H2, H3, H4, H5, H6: MountingHole, MountingHole:MountingHole_3.2mm_M3, symbol Mechanical:MountingHole
- added R3: 4K7, Resistor_THT:R_Axial_DIN0309_L9.0mm_D3.2mm_P12.70mm_Horizontal, symbol Device:R
- added R6, R7: 82, Resistor_THT:R_Axial_DIN0309_L9.0mm_D3.2mm_P12.70mm_Horizontal, symbol Device:R
- added R8, R9: 1K1, Resistor_THT:R_Axial_DIN0309_L9.0mm_D3.2mm_P12.70mm_Horizontal, symbol Device:R
- added SW1, SW2: SW_Push, Button_Switch_THT:SW_PUSH_6mm_H9.5mm, symbol Switch:SW_Push
- D1, D2: footprint LED_SMD:LED_1206_3216Metric_Pad1.42x1.75mm_HandSolder -> LED_THT:LED_D3.0mm
- R1, R2: footprint yabr-main-4:0207_10 -> Resistor_THT:R_Axial_DIN0309_L9.0mm_D3.2mm_P12.70mm_Horizontal
- R4: renamed from R2; value 160 -> 1K1; footprint Resistor_SMD:R_1206_3216Metric_Pad1.30x1.75mm_HandSolder -> Resistor_THT:R_Axial_DIN0309_L9.0mm_D3.2mm_P12.70mm_Horizontal
- R5: renamed from R4; value 160 -> 1K1; footprint Resistor_SMD:R_1206_3216Metric_Pad1.30x1.75mm_HandSolder -> Resistor_THT:R_Axial_DIN0309_L9.0mm_D3.2mm_P12.70mm_Horizontal
- renumbered J3 to J1, U4 to U1, U5 to U2, U2 to U3, U3 to U4
Connections:
- net INT is gone; now on an unnamed net: JP1.8
- net +5V: no longer JP1.1, R4.1, R5.1
- net AD0: now also R3.1
- net GND: now also R3.2, SW1.2, SW2.2
- net VMOT: now also R4.1, R5.1
- net STEP_SELECT_M2: now reaches U4.12 (M2)
- net STEP_SELECT_M2: now also U2.8 (32K_XN/GPIO33/ADC1_CH5), U3.12 (M2)
- net STEP_SELECT_M1: now reaches U4.11 (M1)
- net STEP_SELECT_M1: now also U2.9 (DAC_1/ADC2_CH8/GPIO25), U3.11 (M1)
- net STEP_SELECT_M0: now reaches U4.10 (M0)
- net STEP_SELECT_M0: now also U2.10 (DAC_2/ADC2_CH9/GPIO26), U3.10 (M0)
- net at U3.13 (RST): no longer U3.14 (SLP)
- net STEP_ENABLE: now reaches U3.9 (EN)
- net STEP_ENABLE: now also U2.11 (ADC2_CH7/GPIO27), U4.9 (EN)
- net at U4.13 (RST): no longer U4.14 (SLP)
- net +3V3: now reaches U2.1 (3V3)
- net +3V3: now also JP1.1, R6.1, R7.1, R8.1, R9.1
- net at U2.20 (SD_CLK/GPIO6): now also R8.2, SW1.1
- net at U2.21 (SD_DATA0/GPIO7): now also R9.2, SW2.1
- net at U2.30 (GPIO18): now also D4.1 (K)
- net at U2.31 (GPIO19): now also D3.1 (K)
- net SDL renamed SDA
- new net: D3.2 (A), R6.2
- new net: D4.2 (A), R7.2
Other:
- moved on the sheet: C2, D1, D2, M1, M2, R4, R5, U2, U3, U4
